File: WirelessHeadsetPowerBoard/WirelessHeadsetPowerBoard.kicad_pcb (KiCad board)
At the start: 2 copper layers, 44.4 x 63.5 mm, 44 parts, among them J1 Conn_01x02_Male, J2 Barrel_Jack_MountingPin, J3 Conn_01x02_Female, U1 NXQ1TXH5_101J, Y1 Crystal

Commit message: made changes, made gerbs, winning
Other:
- outline, holes or cut-outs redrawn
