File: WirelessHeadsetPowerBoard/WirelessHeadsetPowerBoard.sch (KiCad schematic (older format))
At the start: 42 parts, among them J1 Conn_01x02_Male, J2 Barrel_Jack_MountingPin, J3 Conn_01x02_Female, U1 NXQ1TXH5_101J, Y1 32.768 kHz Crystal

Commit message: made changes, made gerbs, winning
Parts:
- removed Y1: 32.768 kHz Crystal, Crystal:Crystal_SMD_MicroCrystal_CC7V-T1A-2Pin_3.2x1.5mm_HandSoldering, symbol Device:Crystal_GND23
- added Y1: Crystal, Crystal:Crystal_SMD_MicroCrystal_CC7V-T1A-2Pin_3.2x1.5mm_HandSoldering, symbol Device:Crystal
- D2: footprint LED_SMD:LED_Kingbright_APFA3010_3x1.5mm_Horizontal -> LED_SMD:LED_0603_1608Metric_Pad1.05x0.95mm_HandSolder
Connections:
- net at U1.30 (XTAL_OUT): now also Y1.2
- net at C13.2: now also Y1.1
Changed lines of the file:
@@
 	8650 2850 8650 2525
-$Comp
-L Device:Crystal_GND23 Y1
-U 1 1 601B0393
-P 8925 2950
-F 0 "Y1" H 9119 2996 50  0000 L CNN
-F 1 "32.768 kHz Crystal" H 9100 2850 50  0000 L CNN
-F 2 "Crystal:Crystal_SMD_MicroCrystal_CC7V-T1A-2Pin_3.2x1.5mm_HandSoldering" H 8925 2950 50  0001 C CNN
-F 3 "~" H 8925 2950 50  0001 C CNN
-	1    8925 2950
-	1    0    0    -1
-$EndComp
-Wire Wire Line
-	8925 2600 8925 2750
-$Comp
-L power:GND #PWR020
-U 1 1 601B65FD
-P 9150 2625
-F 0 "#PWR020" H 9150 2375 50  0001 C CNN
-F 1 "GND" H 9155 2452 50  0000 C CNN
-F 2 "" H 9150 2625 50  0001 C CNN
-F 3 "" H 9150 2625 50  0001 C CNN
-	1    9150 2625
-	1    0    0    -1
-$EndComp
 $Comp
 L power:GND #PWR016
@@
 	9350 2525 9350 2950
 Wire Wire Line
-	9350 2950 9075 2950
-Wire Wire Line
 	8650 2525 9350 2525
 Wire Wire Line
-	8925 2600 9150 2600
-Wire Wire Line
-	9150 2600 9150 2625
-Wire Wire Line
 	8775 2950 8750 2950
 Wire Wire Line
@@
 Wire Wire Line
 	8375 2850 8650 2850
-$Comp
-L power:GND #PWR019
-U 1 1 601BD42F
-P 8925 3175
-F 0 "#PWR019" H 8925 2925 50  0001 C CNN
-F 1 "GND" H 8930 3002 50  0000 C CNN
-F 2 "" H 8925 3175 50  0001 C CNN
-F 3 "" H 8925 3175 50  0001 C CNN
-	1    8925 3175
-	1    0    0    -1
-$EndComp
-Wire Wire Line
-	8925 3150 8925 3175
 $Comp
 L power:GND #PWR015
@@
 Wire Wire Line
 	1750 5975 1900 5975
-$Comp
-L Device:C C2
-U 1 1 60276B6A
-P 1900 6175
-F 0 "C2" H 1950 6300 50  0000 L CNN
-F 1 "100nF 50V" H 1975 6075 50  0000 L CNN
-F 2 "Capacitor_SMD:C_0603_1608Metric_Pad1.05x0.95mm_HandSolder" H 1938 6025 50  0001 C CNN
-F 3 "~" H 1900 6175 50  0001 C CNN
-	1    1900 6175
-	1    0    0    -1
-$EndComp
-$Comp
-L Device:C C4
-U 1 1 60276B70
-P 2400 6175
-F 0 "C4" H 2450 6300 50  0000 L CNN
-F 1 "100nF 50V" H 2475 6075 50  0000 L CNN
-F 2 "Capacitor_SMD:C_0603_1608Metric_Pad1.05x0.95mm_HandSolder" H 2438 6025 50  0001 C CNN
-F 3 "~" H 2400 6175 50  0001 C CNN
-	1    2400 6175
-	1    0    0    -1
-$EndComp
-$Comp
-L Device:C C5
-U 1 1 60276B76
-P 2900 6175
-F 0 "C5" H 2950 6300 50  0000 L CNN
-F 1 "82nF 50V" H 2975 6075 50  0000 L CNN
-F 2 "Capacitor_SMD:C_0603_1608Metric_Pad1.05x0.95mm_HandSolder" H 2938 6025 50  0001 C CNN
-F 3 "~" H 2900 6175 50  0001 C CNN
-	1    2900 6175
-	1    0    0    -1
-$EndComp
-$Comp
-L Device:C C6
-U 1 1 60276B7C
-P 3400 6175
-F 0 "C6" H 3450 6300 50  0000 L CNN
-F 1 "82nF 50V" H 3475 6075 50  0000 L CNN
-F 2 "Capacitor_SMD:C_0603_1608Metric_Pad1.05x0.95mm_HandSolder" H 3438 6025 50  0001 C CNN
-F 3 "~" H 3400 6175 50  0001 C CNN
-	1    3400 6175
-	1    0    0    -1
-$EndComp
 Text GLabel 1075 6475 0    50   Output ~ 0
 Coil_Out
@@
 F 0 "D2" H 3675 2025 50  0000 C CNN
 F 1 "LED" H 3550 1975 50  0000 C CNN
-F 2 "LED_SMD:LED_Kingbright_APFA3010_3x1.5mm_Horizontal" H 3675 1925 50  0001 C CNN
+F 2 "LED_SMD:LED_0603_1608Metric_Pad1.05x0.95mm_HandSolder" H 3675 1925 50  0001 C CNN
 F 3 "~" H 3675 1925 50  0001 C CNN
 	1    3675 1925
@@
 Wire Wire Line
 	4025 1925 4025 2050
+$Comp
+L Device:C C6
+U 1 1 60276B7C
+P 3400 6175
+F 0 "C6" H 3450 6300 50  0000 L CNN
+F 1 "82nF 50V" H 3475 6075 50  0000 L CNN
+F 2 "Capacitor_SMD:C_0603_1608Metric_Pad1.05x0.95mm_HandSolder" H 3438 6025 50  0001 C CNN
+F 3 "~" H 3400 6175 50  0001 C CNN
+	1    3400 6175
+	1    0    0    -1
+$EndComp
+$Comp
+L Device:C C5
+U 1 1 60276B76
+P 2900 6175
+F 0 "C5" H 2950 6300 50  0000 L CNN
+F 1 "82nF 50V" H 2975 6075 50  0000 L CNN
+F 2 "Capacitor_SMD:C_0603_1608Metric_Pad1.05x0.95mm_HandSolder" H 2938 6025 50  0001 C CNN
+F 3 "~" H 2900 6175 50  0001 C CNN
+	1    2900 6175
+	1    0    0    -1
+$EndComp
+$Comp
+L Device:C C4
+U 1 1 60276B70
+P 2400 6175
+F 0 "C4" H 2450 6300 50  0000 L CNN
+F 1 "100nF 50V" H 2475 6075 50  0000 L CNN
+F 2 "Capacitor_SMD:C_0603_1608Metric_Pad1.05x0.95mm_HandSolder" H 2438 6025 50  0001 C CNN
+F 3 "~" H 2400 6175 50  0001 C CNN
+	1    2400 6175
+	1    0    0    -1
+$EndComp
+$Comp
+L Device:C C2
+U 1 1 60276B6A
+P 1900 6175
+F 0 "C2" H 1950 6300 50  0000 L CNN
+F 1 "100nF 50V" H 1975 6075 50  0000 L CNN
+F 2 "Capacitor_SMD:C_0603_1608Metric_Pad1.05x0.95mm_HandSolder" H 1938 6025 50  0001 C CNN
+F 3 "~" H 1900 6175 50  0001 C CNN
+	1    1900 6175
+	1    0    0    -1
+$EndComp
+Wire Wire Line
+	9350 2950 9075 2950
+$Comp
+L Device:Crystal Y1
+U 1 1 60337AC3
+P 8925 2950
+F 0 "Y1" H 8925 3218 50  0000 C CNN
+F 1 "Crystal" H 8925 3127 50  0000 C CNN
+F 2 "Crystal:Crystal_SMD_MicroCrystal_CC7V-T1A-2Pin_3.2x1.5mm_HandSoldering" H 8925 2950 50  0001 C CNN
+F 3 "~" H 8925 2950 50  0001 C CNN
+	1    8925 2950
+	1    0    0    -1
+$EndComp
 $EndSCHEMATC
